File: SGP40 Module/SGP40 Module.sch (KiCad schematic (older format))
At the start: 7 parts, among them IC1 SGP40-D-R4, J1 Conn_01x04

Commit message: Cleanup
Parts:
- IC1: footprint SamacSys_Parts:SON80P244X244X95-7N -> SON80P244X244X95-7N
Changed lines of the file:
@@
 $Comp
 L SamacSys_Parts:SGP40-D-R4 IC1
-U 1 1 601335B3
+U 1 1 60135921
 P 5200 3300
 F 0 "IC1" H 5800 3565 50  0000 C CNN
 F 1 "SGP40-D-R4" H 5800 3474 50  0000 C CNN
-F 2 "SamacSys_Parts:SON80P244X244X95-7N" H 6250 3400 50  0001 L CNN
+F 2 "SON80P244X244X95-7N" H 6250 3400 50  0001 L CNN
 F 3 "" H 6250 3300 50  0001 L CNN
 F 4 "Air Quality Sensors Gas Sensor 2.5k pcs IC" H 6250 3200 50  0001 L CNN "Description"
